File: Soil_Moisture_Sensor_SMD-cr.sch (EAGLE design)
At the start: 23 parts, among them IC1 ATMEGA328P

Commit message: 53x20
Parts:
- SL3: device SparkFun-Connectors:M06SIP -> SparkFun-Connectors:M06SMD-1MM
Connections:
- net D0_RX: now also SL3.5; no longer SL3.4
- net D1_TX: now also SL3.6; no longer SL3.5
- net DTR: now also SL3.4; no longer SL3.6
- net GND: now also SL3.3; no longer SL3.1
- net VCC: now also SL3.1; no longer SL3.3
Changed lines of the file:
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@@
 <part name="D1" library="LowPowerLab" deviceset="LED" device="0805" value=""/>
 <part name="SL2" library="SparkFun-Connectors" deviceset="M06" device="SMD-1MM"/>
-<part name="SL3" library="SparkFun-Connectors" deviceset="M06" device="SIP"/>
+<part name="SL3" library="SparkFun-Connectors" deviceset="M06" device="SMD-1MM"/>
 <part name="GND4" library="supply1" deviceset="GND" device=""/>
 <part name="SUPPLY2" library="supply2" deviceset="VCC" device=""/>
@@
 <instance part="GND4" gate="1" x="228.6" y="-17.78" rot="R270"/>
 <instance part="SUPPLY2" gate="G$1" x="223.52" y="-15.24" rot="R90"/>
-<instance part="SUPPLY3" gate="G$1" x="266.7" y="-20.32" rot="R90"/>
+<instance part="SUPPLY3" gate="G$1" x="266.7" y="-15.24" rot="R90"/>
 <instance part="GND5" gate="1" x="259.08" y="-17.78" rot="R270"/>
-<instance part="GND6" gate="1" x="264.16" y="-15.24" rot="R270"/>
+<instance part="GND6" gate="1" x="264.16" y="-20.32" rot="R270"/>
 <instance part="RF1" gate="G$1" x="264.16" y="93.98"/>
 <instance part="SUPPLY4" gate="G$1" x="246.38" y="116.84"/>
@@
 </segment>
 <segment>
-<pinref part="SL3" gate="G$1" pin="2"/>
-<pinref part="GND5" gate="1" pin="GND"/>
-<wire x1="261.62" y1="-17.78" x2="271.78" y2="-17.78" width="0.1524" layer="91"/>
-</segment>
-<segment>
-<pinref part="SL3" gate="G$1" pin="1"/>
-<pinref part="GND6" gate="1" pin="GND"/>
-<wire x1="266.7" y1="-15.24" x2="271.78" y2="-15.24" width="0.1524" layer="91"/>
-</segment>
-<segment>
 <pinref part="RF1" gate="G$1" pin="GND"/>
 <wire x1="251.46" y1="101.6" x2="238.76" y2="101.6" width="0.1524" layer="91"/>
@@
 <pinref part="GND3" gate="1" pin="GND"/>
 <wire x1="-66.04" y1="-35.56" x2="-66.04" y2="-43.18" width="0.1524" layer="91"/>
+</segment>
+<segment>
+<pinref part="GND5" gate="1" pin="GND"/>
+<pinref part="SL3" gate="G$1" pin="2"/>
+<wire x1="261.62" y1="-17.78" x2="271.78" y2="-17.78" width="0.1524" layer="91"/>
+</segment>
+<segment>
+<pinref part="GND6" gate="1" pin="GND"/>
+<pinref part="SL3" gate="G$1" pin="3"/>
+<wire x1="266.7" y1="-20.32" x2="271.78" y2="-20.32" width="0.1524" layer="91"/>
 </segment>
 </net>
@@
 </segment>
 <segment>
-<pinref part="SL3" gate="G$1" pin="3"/>
-<wire x1="271.78" y1="-20.32" x2="269.24" y2="-20.32" width="0.1524" layer="91"/>
-<pinref part="SUPPLY3" gate="G$1" pin="VCC"/>
-</segment>
-<segment>
 <pinref part="RF1" gate="G$1" pin="3V"/>
 <pinref part="SUPPLY4" gate="G$1" pin="VCC"/>
@@
 <wire x1="-53.34" y1="-5.08" x2="-53.34" y2="-7.62" width="0.1524" layer="91"/>
 </segment>
+<segment>
+<pinref part="SUPPLY3" gate="G$1" pin="VCC"/>
+<pinref part="SL3" gate="G$1" pin="1"/>
+<wire x1="269.24" y1="-15.24" x2="271.78" y2="-15.24" width="0.1524" layer="91"/>
+</segment>
 </net>
 <net name="DTR" class="0">
@@
 </segment>
 <segment>
-<pinref part="SL3" gate="G$1" pin="6"/>
-<wire x1="271.78" y1="-27.94" x2="254" y2="-27.94" width="0.1524" layer="91"/>
-<label x="254" y="-27.94" size="1.778" layer="95" rot="MR0"/>
+<pinref part="SL3" gate="G$1" pin="4"/>
+<wire x1="271.78" y1="-22.86" x2="254" y2="-22.86" width="0.1524" layer="91"/>
+<label x="254" y="-22.86" size="1.778" layer="95" rot="MR0"/>
 </segment>
 </net>
@@
 <net name="D0_RX" class="0">
 <segment>
-<pinref part="SL3" gate="G$1" pin="4"/>
-<wire x1="271.78" y1="-22.86" x2="254" y2="-22.86" width="0.1524" layer="91"/>
-<label x="254" y="-22.86" size="1.778" layer="95" rot="MR0"/>
+<pinref part="SL3" gate="G$1" pin="5"/>
+<wire x1="271.78" y1="-25.4" x2="254" y2="-25.4" width="0.1524" layer="91"/>
+<label x="254" y="-25.4" size="1.778" layer="95" rot="MR0"/>
 </segment>
 <segment>
@@
 <net name="D1_TX" class="0">
 <segment>
-<pinref part="SL3" gate="G$1" pin="5"/>
-<wire x1="271.78" y1="-25.4" x2="254" y2="-25.4" width="0.1524" layer="91"/>
-<label x="254" y="-25.4" size="1.778" layer="95" rot="MR0"/>
+<pinref part="SL3" gate="G$1" pin="6"/>
+<wire x1="271.78" y1="-27.94" x2="254" y2="-27.94" width="0.1524" layer="91"/>
+<label x="254" y="-27.94" size="1.778" layer="95" rot="MR0"/>
 </segment>
 <segment>
@@
 </segment>
 </net>
-<net name="N$3" class="0">
+<net name="N$3" class="1">
 <segment>
 <pinref part="J1" gate="G$1" pin="2"/>
@@
 </segment>
 </net>
-<net name="N$5" class="0">
+<net name="N$5" class="1">
 <segment>
 <pinref part="IC1" gate="G$1" pin="PC1(ADC1)"/>

Commit message: pcb-v1.1.3
Parts:
- LED1: device led:LED3MM -> led:LED5MM
Changed lines of the file:
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@@
 <part name="C4" library="LowPowerLab" deviceset="CAP" device="0805-CAP" value="0.1uF"/>
 <part name="J1" library="SparkFun-Connectors" deviceset="CONN_02" device=""/>
-<part name="LED1" library="led" deviceset="LED" device="3MM"/>
+<part name="LED1" library="led" deviceset="LED" device="5MM"/>
 <part name="R5" library="LowPowerLab" deviceset="RESISTOR" device="0805-RES" value="1k5"/>
 <part name="FRAME1" library="frames" deviceset="A3L-LOC" device=""/>

Commit message: pcb-v1.1.3
Other:
- note added: "V1.1.3"
- note removed: "V1.1.2a"
Changed lines of the file:
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@@
 <wire x1="-86.106" y1="29.718" x2="-27.686" y2="29.718" width="0.4064" layer="94" style="longdash"/>
 <text x="-76.2" y="22.86" size="2.54" layer="94">Measuring Battery Level</text>
-<text x="281.94" y="-91.44" size="2.54" layer="94">V1.1.2a</text>
+<text x="281.94" y="-91.44" size="2.54" layer="94">V1.1.3</text>
 </plain>
 <instances>
